File: Hardware/Schematics/ProTag.kicad_pcb (KiCad board)
At the start: 2 copper layers, 24 x 24 mm, 56 parts, among them IC1 MC3216, IC2 QN9090THN_001Z, J1 Conn_01x01_Female, J10 TEST_POINT, J11 TEST_POINT, J12 TEST_POINT, J13 TEST_POINT, J14 TEST_POINT, J15 TEST_POINT, J16 TEST_POINT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

Commit message: Add files via upload
Parts:
- D1, D2, R4, R7, Y2: moved to B.Cu
- moved R9 108.9 mm to (59.1, 41.3)
- moved R8 96.7 mm to (63.9, 42.0), turned to 180 degrees
- moved Q1 81.6 mm to (61.5, 42.0)
- moved C8 51.9 mm to (135.5, 90.2), turned to 90 degrees
- moved R7 51.1 mm to (131.4, 86.5), turned to 180 degrees
- moved J7 49.4 mm to (133.8, 92.9)
- moved C2 48.5 mm to (129.9, 91.0)
- moved U1 48.4 mm to (142.9, 103.0)
- moved C1 47.3 mm to (140.4, 102.6), turned to 90 degrees
- moved C5 45.1 mm to (145.2, 104.1), turned to 90 degrees
- moved IC1 44.9 mm to (132.9, 90.5)
- moved J8 44.4 mm to (135.9, 92.9)
- moved J17 44.4 mm to (170.3, 26.8)
- moved J18 44.4 mm to (173.3, 26.8)
- moved C14 44.4 mm to (182.8, 19.9)
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Routing:
- net BUTTON_1: track 0.00 -> 19.7 mm, vias 0 -> 1
- net SDA: track 0.00 -> 16.8 mm
- net GND: track 0.77 -> 15.4 mm, vias 1 -> 5
- net SCL: track 0.00 -> 12.5 mm
- net INTN: track 0.00 -> 12.2 mm
- net LED_1: track 0.00 -> 7.25 mm, vias 0 -> 1
- net Net-(C12-Pad1): track 2.30 -> 9.42 mm, vias 0 -> 2
- net LA: track 0.00 -> 6.32 mm
- net LB: track 0.00 -> 5.70 mm
- net +3V3: track 2.95 -> 8.48 mm
- net LED_2: track 0.00 -> 3.08 mm, vias 0 -> 1
- net ANT: track 4.15 -> 1.66 mm
- net XTAL32_N: track 3.54 -> 5.84 mm
- net Net-(IC2-Pad29): track 3.10 -> 5.03 mm
- net Net-(C6-Pad1): track 0.00 -> 1.93 mm
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Other:
- board size 24 x 24 mm -> 30 x 30 mm

Commit message: Add files via upload
Parts:
- removed D1: LED, Diode_SMD:D_0201_0603Metric
- removed J1: Conn_01x01_Female, TestPoint:TestPoint_Pad_D1.0mm
- removed R4: 1.5K, Resistor_SMD:R_0201_0603Metric
- added ANT1: 2450AT18B100E, ASSETS:ANTC3216X140N, F.Cu at (170.8, 107.3)
- added G***: LOGO, ASSETS:company_l1, F.Cu at (176.9, 109.4)
- J10, J11, J12, J13, J14, J15, J16, J17, J18, J19, J2, J3, J4, J5, J6, J7, J8, J9: footprint TestPoint:TestPoint_Pad_D1.0mm -> ASSETS:testpoint_0.3mm
- Q1, R8, R9: moved to B.Cu
- moved R9 155.4 mm to (188.0, 128.1), turned to 90 degrees
- moved Q1 154.5 mm to (190.1, 127.5)
- moved R8 154.0 mm to (191.3, 128.6), turned to 90 degrees
- moved C9 117.0 mm to (192.2, 127.9), turned to 180 degrees
- moved J19 112.6 mm to (190.5, 127.0), turned to 90 degrees
- moved J2 110.2 mm to (187.0, 124.5), turned to 90 degrees
- moved J3 110.0 mm to (186.6, 121.4), turned to 90 degrees
- moved J18 101.8 mm to (191.6, 127.0), turned to 90 degrees
- moved J13 101.7 mm to (192.6, 112.9)
- moved J10 100.7 mm to (188.2, 118.4), turned to 180 degrees
- moved J12 99.7 mm to (192.6, 113.7), turned to 180 degrees
- moved J6 99.6 mm to (186.9, 123.7), turned to 270 degrees
- moved J14 97.8 mm to (193.1, 114.4)
- moved J11 96.3 mm to (189.0, 118.4)
- moved R3 95.0 mm to (193.4, 113.3), turned to 90 degrees
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Connections:
- IC2 pad 7: LED_2 -> Net-(IC2-Pad7)
Routing:
- net +3V3: track 8.48 -> 32.2 mm, vias 0 -> 5
- net GND: track 15.4 -> 34.1 mm, vias 5 -> 17
- net SCL: track 12.5 -> 27.7 mm, vias 0 -> 2
- net INTN: track 12.2 -> 26.3 mm
- net VDD: track 0.00 -> 13.8 mm, vias 0 -> 3
- net NPN_CNTL: track 0.00 -> 13.7 mm, vias 0 -> 1
- net Net-(ANT1-Pad1): track 1.93 -> 14.4 mm
- net SDA: track 16.8 -> 23.9 mm, vias 0 -> 2
- net ON_OFF: track 0.00 -> 6.74 mm, vias 0 -> 1
- net Net-(C12-Pad1): track 9.42 -> 15.0 mm, vias 2 -> 0
- net BUTTON_1: track 19.7 -> 15.6 mm
- net LED_2: track 3.08 -> 0.00 mm, vias 1 -> 0
- net Net-(IC2-Pad29): track 5.03 -> 2.56 mm
- net SWDIO: track 0.00 -> 2.05 mm
- net RSTN: track 0.00 -> 2.05 mm
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- added copper zone on F.Cu, net +3V3
- added copper zone on B.Cu, net GND
Other:
- outline, holes or cut-outs redrawn
- board text added: "ProTag v1 09.05.2021"
